File: 3v3LipoChargeBoost.kicad_sch (KiCad schematic)
At the start: 14 parts, among them J1 BATT, J2 USB_B_Mini, J3 Output, SW1 Power->, U1 TPS63001, U2 MCP73831-2-OT

Commit message: Update 3v3LipoChargeBoost.kicad_sch
Parts:
- removed SW1: Power->, SnapEDA Library:3pin_switch, symbol Switch:SW_Push
Changed lines of the file:
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@@
   (junction (at 57.15 26.67) (diameter 0) (color 0 0 0 0)
-  )
-  (junction (at 81.28 52.07) (diameter 0) (color 0 0 0 0)
   )
   (junction (at 60.96 68.58) (diameter 0) (color 0 0 0 0)
@@
   (text "MCP1661 as applicable \n5 pin boost IC" (at 72.39 39.37 0)
     (effects (font (size 1.27 1.27)) (justify left bottom))
-  )
-  (global_label "BATT" (shape input) (at 71.12 52.07 180) (fields_autoplaced)
-    (effects (font (size 1.27 1.27)) (justify right))
-    (property "Intersheet References" "${INTERSHEET_REFS}" (id 0) (at 0 0 0)
-      (effects (font (size 1.27 1.27)) hide)
-    )
   )
   (global_label "BATT" (shape input) (at 27.94 26.67 180) (fields_autoplaced)
@@
     (pin "1")
   )
-  (symbol (lib_id "Switch:SW_Push") (at 76.2 52.07 180) (unit 1)
-    (in_bom yes) (on_board yes)
-    (property "Reference" "SW1" (id 0) (at 76.2 59.309 0)
-      (effects (font (size 1.27 1.27)) hide)
-    )
-    (property "Value" "Power->" (id 1) (at 76.2 56.9976 0)
-      (effects (font (size 1.27 1.27)) hide)
-    )
-    (property "Footprint" "SnapEDA Library:3pin_switch" (id 2) (at 76.2 57.15 0)
-      (effects (font (size 1.27 1.27)) hide)
-    )
-    (property "Datasheet" "~" (id 3) (at 76.2 57.15 0)
-      (effects (font (size 1.27 1.27)) hide)
-    )
-    (pin "1")
-    (pin "2")
-  )
   (symbol (lib_id "Battery_Management:MCP73831-2-OT") (at 60.96 60.96 0) (unit 1)
     (in_bom yes) (on_board yes)
@@
       (reference "R2") (unit 1) (value "2k") (footprint "Resistor_SMD:R_1206_3216Metric")
     )
-    (path "/00000000-0000-0000-0000-00006123fd29"
-      (reference "SW1") (unit 1) (value "Power->") (footprint "SnapEDA Library:3pin_switch")
-    )
     (path "/00000000-0000-0000-0000-000061234420"
